File: hardware/com-gnd-scale_v0.0.1/com-gnd-scale_v0.0.1.kicad_sch (KiCad schematic)
At the start: 5 parts

Commit message: Update com-gnd-scale_v0.0.1.kicad_sch
Other:
- note added: "Force Sensors"
- note added: "SPDT Switch"
Changed lines of the file:
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@@
+    (stroke (width 0) (type default) (color 0 0 0 0))
+  )
+  (wire (pts (xy 166.37 49.53) (xy 173.99 49.53))
     (stroke (width 0) (type default) (color 0 0 0 0))
   )
@@
     (stroke (width 0) (type default) (color 0 0 0 0))
   )
+  (wire (pts (xy 166.37 45.72) (xy 173.99 45.72))
+    (stroke (width 0) (type default) (color 0 0 0 0))
+  )
+  (wire (pts (xy 31.75 107.95) (xy 62.23 107.95))
+    (stroke (width 0) (type default) (color 0 0 0 0))
+  )
   (wire (pts (xy 271.78 64.77) (xy 166.37 64.77))
     (stroke (width 0) (type default) (color 0 0 0 0))
@@
     (stroke (width 0) (type default) (color 0 0 0 0))
   )
+  (wire (pts (xy 97.79 107.95) (xy 72.39 107.95))
+    (stroke (width 0) (type default) (color 0 0 0 0))
+  )
   (wire (pts (xy 271.78 45.72) (xy 271.78 64.77))
     (stroke (width 0) (type default) (color 0 0 0 0))
@@
     (stroke (width 0) (type default) (color 0 0 0 0))
   )
+  (wire (pts (xy 62.23 107.95) (xy 62.23 92.71))
+    (stroke (width 0) (type default) (color 0 0 0 0))
+  )
   (wire (pts (xy 186.69 80.01) (xy 166.37 80.01))
     (stroke (width 0) (type default) (color 0 0 0 0))
@@
     (stroke (width 0) (type default) (color 0 0 0 0))
   )
+  (wire (pts (xy 31.75 144.78) (xy 31.75 107.95))
+    (stroke (width 0) (type default) (color 0 0 0 0))
+  )
   (wire (pts (xy 186.69 91.44) (xy 186.69 80.01))
     (stroke (width 0) (type default) (color 0 0 0 0))
@@
     (stroke (width 0) (type default) (color 0 0 0 0))
   )
+  (wire (pts (xy 97.79 142.24) (xy 97.79 107.95))
+    (stroke (width 0) (type default) (color 0 0 0 0))
+  )
+  (wire (pts (xy 72.39 107.95) (xy 72.39 92.71))
+    (stroke (width 0) (type default) (color 0 0 0 0))
+  )
   (wire (pts (xy 101.6 64.77) (xy 119.38 64.77))
     (stroke (width 0) (type default) (color 0 0 0 0))
   )
-  (wire (pts (xy 38.1 144.78) (xy 52.07 144.78))
-    (stroke (width 0) (type default) (color 0 0 0 0))
-  )
-  (wire (pts (xy 80.01 142.24) (xy 90.17 142.24))
+  (wire (pts (xy 31.75 144.78) (xy 52.07 144.78))
+    (stroke (width 0) (type default) (color 0 0 0 0))
+  )
+  (wire (pts (xy 80.01 142.24) (xy 97.79 142.24))
     (stroke (width 0) (type default) (color 0 0 0 0))
   )
@@
   (wire (pts (xy 236.22 57.15) (xy 166.37 57.15))
     (stroke (width 0) (type default) (color 0 0 0 0))
+  )
+  (text "SPDT Switch" (at 60.96 121.92 0)
+    (effects (font (size 1.27 1.27)) (justify left bottom))
+  )
+  (text "Force Sensors" (at 231.14 29.21 0)
+    (effects (font (size 1.27 1.27)) (justify left bottom))
   )
   (text "GOM GND Scale v0.0.1\n" (at 189.23 190.5 0)
@@
     (effects (font (size 1.27 1.27)) (justify right bottom))
   )
+  (label "Exc2" (at 168.91 49.53 0)
+    (effects (font (size 1.27 1.27)) (justify left bottom))
+  )
   (label "EXCEN" (at 90.17 142.24 180)
     (effects (font (size 1.524 1.524)) (justify right bottom))
@@
   )
   (label "Exc2" (at 262.89 50.8 0)
+    (effects (font (size 1.27 1.27)) (justify left bottom))
+  )
+  (label "Exc1" (at 168.91 45.72 0)
     (effects (font (size 1.27 1.27)) (justify left bottom))
   )
@@
       (effects (font (size 1.27 1.27)) (justify left))
     )
-    (pin "GPIO26" input (at 30.48 72.39 180)
-      (effects (font (size 1.27 1.27)) (justify left))
-    )
-    (pin "GPIO25" input (at 30.48 68.58 180)
-      (effects (font (size 1.27 1.27)) (justify left))
-    )
+    (pin "GPIO26" input (at 72.39 92.71 270)
+      (effects (font (size 1.27 1.27)) (justify left))
+    )
+    (pin "GPIO25" input (at 62.23 92.71 270)
+      (effects (font (size 1.27 1.27)) (justify left))
+    )

Commit message: Fix voltage level on excitation h-bridge pwr. More modifications for isolated testing on the refrev issue.
Connections:
- net +4V: no longer IC?.1 (V+)
- net GNDA: no longer IC?.6 (GND)
- new net +5V: IC?.1 (V+)
- new net GND: IC?.6 (GND)
Changed lines of the file:
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@@
+    (stroke (width 0) (type default) (color 0 0 0 0))
+  )
+  (wire (pts (xy 114.3 34.29) (xy 119.38 34.29))
     (stroke (width 0) (type default) (color 0 0 0 0))
   )
@@
   )
   (wire (pts (xy 101.6 57.15) (xy 119.38 57.15))
+    (stroke (width 0) (type default) (color 0 0 0 0))
+  )
+  (wire (pts (xy 114.3 38.1) (xy 119.38 38.1))
     (stroke (width 0) (type default) (color 0 0 0 0))
   )
@@
     (property "Datasheet" "" (id 3) (at 52.07 139.7 0)
       (effects (font (size 1.27 1.27)) hide)
+    )
+    (pin "1")
+  )
+  (symbol (lib_id "ESP32-DevKit-Lipo_Rev_C:GND") (at 114.3 38.1 270) (unit 1)
+    (in_bom yes) (on_board yes) (fields_autoplaced)
+    (property "Reference" "#PWR?" (id 0) (at 107.95 38.1 0)
+      (effects (font (size 1.27 1.27)) hide)
+    )
+    (property "Value" "GND" (id 1) (at 110.49 38.0999 90)
+      (effects (font (size 1.27 1.27)) (justify right))
+    )
+    (property "Footprint" "" (id 2) (at 114.3 38.1 0)
+      (effects (font (size 1.524 1.524)))
+    )
+    (property "Datasheet" "" (id 3) (at 114.3 38.1 0)
+      (effects (font (size 1.524 1.524)))
     )
     (pin "1")
@@
     (pin "1")
   )
-  (symbol (lib_id "BB-ADS1262-Rev.A:GNDA") (at 80.01 147.32 0) (mirror y) (unit 1)
+  (symbol (lib_id "ESP32-DevKit-Lipo_Rev_C:GND") (at 80.01 147.32 0) (unit 1)
     (in_bom yes) (on_board yes)
     (property "Reference" "#PWR?" (id 0) (at 80.01 153.67 0)
       (effects (font (size 1.27 1.27)) hide)
     )
-    (property "Value" "GNDA" (id 1) (at 79.883 151.7142 0))
+    (property "Value" "GND" (id 1) (at 80.01 152.4 0))
     (property "Footprint" "" (id 2) (at 80.01 147.32 0)
       (effects (font (size 1.524 1.524)))
     )
     (property "Datasheet" "" (id 3) (at 80.01 147.32 0)
+      (effects (font (size 1.524 1.524)))
+    )
+    (pin "1")
+  )
+  (symbol (lib_id "ESP32-DevKit-Lipo_Rev_C:+5V") (at 52.07 137.16 0) (unit 1)
+    (in_bom yes) (on_board yes) (fields_autoplaced)
+    (property "Reference" "#PWR?" (id 0) (at 52.07 140.97 0)
+      (effects (font (size 1.27 1.27)) hide)
+    )
+    (property "Value" "+5V" (id 1) (at 52.07 132.08 0))
+    (property "Footprint" "" (id 2) (at 52.07 137.16 0)
+      (effects (font (size 1.524 1.524)))
+    )
+    (property "Datasheet" "" (id 3) (at 52.07 137.16 0)
       (effects (font (size 1.524 1.524)))
     )
@@
     (pin "1")
   )
+  (symbol (lib_id "ESP32-DevKit-Lipo_Rev_C:+3.3V") (at 114.3 34.29 90) (unit 1)
+    (in_bom yes) (on_board yes) (fields_autoplaced)
+    (property "Reference" "#PWR?" (id 0) (at 118.11 34.29 0)
+      (effects (font (size 1.27 1.27)) hide)
+    )
+    (property "Value" "+3.3V" (id 1) (at 110.49 34.2899 90)
+      (effects (font (size 1.27 1.27)) (justify left))
+    )
+    (property "Footprint" "" (id 2) (at 114.3 34.29 0)
+      (effects (font (size 1.524 1.524)))
+    )
+    (property "Datasheet" "" (id 3) (at 114.3 34.29 0)
+      (effects (font (size 1.524 1.524)))
+    )
+    (pin "1")
+  )
   (symbol (lib_id "BB-ADS1262-Rev.A:GNDA") (at 52.07 147.32 0) (mirror y) (unit 1)
     (in_bom yes) (on_board yes)
@@
     (pin "3")
     (pin "4")
-  )
-  (symbol (lib_id "power:+4VA") (at 52.07 137.16 0) (unit 1)
-    (in_bom yes) (on_board yes) (fields_autoplaced)
-    (property "Reference" "#PWR?" (id 0) (at 52.07 140.97 0)
-      (effects (font (size 1.27 1.27)) hide)
-    )
-    (property "Value" "+4VA" (id 1) (at 52.07 132.08 0))
-    (property "Footprint" "" (id 2) (at 52.07 137.16 0)
-      (effects (font (size 1.27 1.27)) hide)
-    )
-    (property "Datasheet" "" (id 3) (at 52.07 137.16 0)
-      (effects (font (size 1.27 1.27)) hide)
-    )
-    (pin "1")
   )
   (symbol (lib_id "power:GNDA") (at 115.57 49.53 270) (unit 1)
@@
       (reference "#PWR?") (unit 1) (value "+4VA") (footprint "")
     )
+    (path "/5fc2cbfd-e4f9-4e12-9640-1ee785166b8c"
+      (reference "#PWR?") (unit 1) (value "GND") (footprint "")
+    )
     (path "/83505d28-20e8-41e6-9315-c348e240e9e0/8266e410-5a80-4ffa-b151-31c825bcb7cf"
       (reference "#PWR?") (unit 1) (value "+4VA") (footprint "")
@@
       (reference "#PWR?") (unit 1) (value "GNDA") (footprint "")
     )
-    (path "/b2fc8c30-9639-46bc-8270-cd17328fef5a"
-      (reference "#PWR?") (unit 1) (value "GNDA") (footprint "")
+    (path "/9e321569-1454-43aa-97b2-3a9d88a70a1c"
+      (reference "#PWR?") (unit 1) (value "GND") (footprint "")
+    )
+    (path "/af541b7f-47e2-4338-86d3-64a72b5b7aba"
+      (reference "#PWR?") (unit 1) (value "+5V") (footprint "")
     )
     (path "/bb0096c1-baaf-48be-85a8-182ffe204862"
@@
       (reference "#PWR?") (unit 1) (value "+4VA") (footprint "")
     )
+    (path "/daf121ec-2c00-4e96-96aa-2bc6f7a0fed5"
+      (reference "#PWR?") (unit 1) (value "+3.3V") (footprint "")
+    )
     (path "/dd594143-20c7-496d-a3a0-136ae5aa72e8"
       (reference "#PWR?") (unit 1) (value "GNDA") (footprint "")
     )
-    (path "/e0e3fa98-f2cd-47f2-be2d-0635272b0474"
-      (reference "#PWR?") (unit 1) (value "+4VA") (footprint "")
-    )
     (path "/fa84dcfa-c418-458c-8529-5a704eb514f4"
